File: FXTal_no_holes.kicad_sch (KiCad schematic)
At the start: 150 parts, among them J1 CONN_CAP_IBM_F

Commit message: push
Parts:
- removed H1, H10, H11, H12, H13, H14, H15, H16, H17, H18, H19, H2, H20, H21, H22, H23, H24, H25, H26, H27, H28, H29, H3, H30, H31, H32, H4, H5, H6, H7, H8, H9: HOLE, lib_fp:HOLE, symbol lib_sch:HOLE
- SW_0: value 0 -> 8,7; footprint lib_fp:SW_CAP_IBM_F -> lib_fp:SW_CAP_IBM_F_ALT
- SW_02: value 2 -> 3,8
- SW_03: value 3 -> 4,7
- SW_04: value 4 -> 4,8
- SW_05: value 5 -> 5,7
- SW_06: value 6 -> 5,8
- SW_07: value 7 -> 6,8
- SW_08: value 8 -> 7,7; footprint lib_fp:SW_CAP_IBM_F -> lib_fp:SW_CAP_IBM_F_ALT
- SW_09: value 9 -> 7,8; footprint lib_fp:SW_CAP_IBM_F_ALT -> lib_fp:SW_CAP_IBM_F
- SW_1: value 1 -> 2,8; footprint lib_fp:SW_CAP_IBM_F_ALT -> lib_fp:SW_CAP_IBM_F
- SW_10: value A -> 3,4
- SW_11: value B -> 6,2
- SW_12: value BSLS -> A,6; footprint lib_fp:SW_CAP_IBM_F -> lib_fp:SW_CAP_IBM_F_ALT
- SW_13: value BSPC -> A,8
- SW_14: value C -> 4,4
- SW_15: value CAPS -> 2,5; footprint lib_fp:SW_CAP_IBM_F_ALT -> lib_fp:SW_CAP_IBM_F
- SW_16: value COMM -> 7,3
- SW_17: value D -> 4,5; footprint lib_fp:SW_CAP_IBM_F_ALT -> lib_fp:SW_CAP_IBM_F
- SW_18: value DOT -> 8,2
- SW_19: value E -> 4,6
- SW_20: value ENT -> A,4
- SW_21: value EQL -> 9,8; footprint lib_fp:SW_CAP_IBM_F -> lib_fp:SW_CAP_IBM_F_ALT
- SW_22: value GRV -> 2,7; footprint lib_fp:SW_CAP_IBM_F -> lib_fp:SW_CAP_IBM_F_ALT
- SW_23: value F2 -> 2,1
- SW_24: value F -> 5,4; footprint lib_fp:SW_CAP_IBM_F -> lib_fp:SW_CAP_IBM_F_ALT
- SW_25: value F9 -> 1,7; footprint lib_fp:SW_CAP_IBM_F -> lib_fp:SW_CAP_IBM_F_ALT
- SW_26: value F10 -> 1,8; footprint lib_fp:SW_CAP_IBM_F_ALT -> lib_fp:SW_CAP_IBM_F
- SW_27: value F7 -> 1,5; footprint lib_fp:SW_CAP_IBM_F -> lib_fp:SW_CAP_IBM_F_ALT
- SW_28: value F8 -> 1,6; footprint lib_fp:SW_CAP_IBM_F_ALT -> lib_fp:SW_CAP_IBM_F
- SW_29: value F5 -> 1,3; footprint lib_fp:SW_CAP_IBM_F -> lib_fp:SW_CAP_IBM_F_ALT
- SW_30: value F6 -> 1,4; footprint lib_fp:SW_CAP_IBM_F_ALT -> lib_fp:SW_CAP_IBM_F
- SW_31: value F3 -> 1,2; footprint lib_fp:SW_CAP_IBM_F -> lib_fp:SW_CAP_IBM_F_ALT
- SW_32: value F4 -> 2,3
- SW_33: value F1 -> 1,1; footprint lib_fp:SW_CAP_IBM_F -> lib_fp:SW_CAP_IBM_F_ALT
- SW_34: value FN -> 4,2; footprint lib_fp:SW_CAP_IBM_F_ALT -> lib_fp:SW_CAP_IBM_F
- SW_35: value G -> 5,3; footprint lib_fp:SW_CAP_IBM_F_ALT -> lib_fp:SW_CAP_IBM_F
- SW_36: value H -> 6,4; footprint lib_fp:SW_CAP_IBM_F -> lib_fp:SW_CAP_IBM_F_ALT
- SW_37: value I -> 7,5
- SW_38: value J -> 6,5; footprint lib_fp:SW_CAP_IBM_F_ALT -> lib_fp:SW_CAP_IBM_F
- SW_39: value K -> 7,4; footprint lib_fp:SW_CAP_IBM_F -> lib_fp:SW_CAP_IBM_F_ALT
- SW_40: value L -> 8,4
- SW_41: value LALT -> 4,1; footprint lib_fp:SW_CAP_IBM_F -> lib_fp:SW_CAP_IBM_F_ALT
- SW_42: value LBRC -> 9,6
- SW_43: value LCTL -> 2,2; footprint lib_fp:SW_CAP_IBM_F_ALT -> lib_fp:SW_CAP_IBM_F
- SW_44: value LGUI -> 3,1; footprint lib_fp:SW_CAP_IBM_F -> lib_fp:SW_CAP_IBM_F_ALT
- SW_45: value LSFT -> 2,4; footprint lib_fp:SW_CAP_IBM_F_ALT -> lib_fp:SW_CAP_IBM_F
- SW_46: value M -> 7,2; footprint lib_fp:SW_CAP_IBM_F -> lib_fp:SW_CAP_IBM_F_ALT
- SW_47: value MINS -> 8,8; footprint lib_fp:SW_CAP_IBM_F_ALT -> lib_fp:SW_CAP_IBM_F
- SW_48: value N -> 6,3
- SW_49: value NUBS -> 3,3; footprint lib_fp:SW_CAP_IBM_F -> lib_fp:SW_CAP_IBM_F_ALT
- SW_50: value NUHS -> 9,5
- SW_51: value O -> 7,6
- SW_52: value OPEN -> 9,1
- SW_53: value P10 -> B,5
- SW_54: value P11 -> C,4; footprint lib_fp:SW_CAP_IBM_F -> lib_fp:SW_CAP_IBM_F_ALT
- SW_55: value P12 -> C,3; footprint lib_fp:SW_CAP_IBM_F_ALT -> lib_fp:SW_CAP_IBM_F
- SW_56: value P5 -> A,3
- SW_57: value P6 -> B,4
- SW_58: value P7 -> B,3; footprint lib_fp:SW_CAP_IBM_F_ALT -> lib_fp:SW_CAP_IBM_F
- SW_59: value P8 -> C,2
- SW_60: value P1 -> A,1
- SW_61: value P2 -> B,1
- SW_62: value P3 -> B,2
- SW_63: value P17 -> B,8
- SW_64: value P4 -> C,1; footprint lib_fp:SW_CAP_IBM_F_ALT -> lib_fp:SW_CAP_IBM_F
- SW_65: value P -> 8,6; footprint lib_fp:SW_CAP_IBM_F_ALT -> lib_fp:SW_CAP_IBM_F
- SW_66: value P18 -> B,7
- SW_67: value P19 -> C,8
- SW_68: value P20 -> C,7
- SW_69: value P13 -> A,7
- SW_70: value P14 -> B,6
- SW_71: value P15 -> C,6
- SW_72: value P16 -> C,5
- SW_73: value P9 -> A,5
- SW_74: value Q -> 3,6; footprint lib_fp:SW_CAP_IBM_F -> lib_fp:SW_CAP_IBM_F_ALT
- SW_75: value QUOT -> 9,4
- SW_76: value R -> 5,5
- SW_77: value RALT -> 8,1
- SW_78: value RBRC -> 9,7; footprint lib_fp:SW_CAP_IBM_F_ALT -> lib_fp:SW_CAP_IBM_F
- SW_79: value RCTL -> 9,2
- SW_80: value RGUI -> 9,1; footprint lib_fp:SW_CAP_IBM_F -> lib_fp:SW_CAP_IBM_F_ALT
- SW_81: value RSFT -> 9,3
- SW_82: value RSFT -> A,2
- SW_83: value S -> 3,5
- SW_84: value SCLN -> 8,5
- SW_85: value SLSH -> 8,3
- SW_86: value SPC1 -> 5,1; footprint lib_fp:SW_CAP_IBM_F_ALT -> lib_fp:SW_CAP_IBM_F
- SW_87: value SPC2 -> 7,1; footprint lib_fp:SW_CAP_IBM_F -> lib_fp:SW_CAP_IBM_F_ALT
- SW_88: value SPC -> 6,1
- SW_89: value T -> 5,6
- SW_90: value TAB -> 2,6
- SW_91: value U -> 6,6; footprint lib_fp:SW_CAP_IBM_F_ALT -> lib_fp:SW_CAP_IBM_F
- SW_92: value V -> 5,2; footprint lib_fp:SW_CAP_IBM_F -> lib_fp:SW_CAP_IBM_F_ALT
- SW_93: value W -> 3,7
- SW_94: value X -> 4,3
- SW_95: value Y -> 6,7; footprint lib_fp:SW_CAP_IBM_F -> lib_fp:SW_CAP_IBM_F_ALT
- SW_96: value Z -> 3,2; footprint lib_fp:SW_CAP_IBM_F_ALT -> lib_fp:SW_CAP_IBM_F
