File: FXTal_rev1.kicad_pcb (KiCad board)
At the start: 2 copper layers, 418.9 x 150.2 mm, 118 parts, among them J1 CONN_CAP_IBM_F

Commit message: changes to wireing
Parts:
- moved SW_43 0.66 mm to (110.8, 269.0)
- moved COL_9_TP17 0.17 mm to (345.3, 279.8)
- moved COL_5_TP13 0.17 mm to (208.5, 279.0)
- moved SW_20 0.17 mm to (367.4, 227.0)
- moved SW_57 0.17 mm to (405.5, 248.0)
- moved SW_68 0.17 mm to (443.5, 185.0)
- moved SW_70 0.17 mm to (405.4, 206.0)
- moved COL_2_TP10 0.17 mm to (82.4, 279.0)
- moved COL_6_TP14 0.17 mm to (235.2, 279.2)
- moved COL_A_TP18 0.17 mm to (382.1, 279.0)
- moved COL_B_TP19 0.17 mm to (409.8, 279.8)
- moved COL_C_TP20 0.17 mm to (439.5, 279.0)
- moved SW_02 0.17 mm to (144.0, 185.0)
- moved SW_03 0.17 mm to (163.0, 185.0)
- moved SW_04 0.17 mm to (182.0, 185.0)
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Routing:
- net COL_2: track 411.3 -> 424.0 mm
- net COL_5: track 302.1 -> 314.5 mm
- net COL_4: track 344.3 -> 355.3 mm
- net COL_7: track 259.4 -> 269.2 mm
- net COL_1: track 431.3 -> 439.0 mm
- net COL_6: track 279.2 -> 281.9 mm
- net COL_3: track 369.5 -> 367.9 mm
- net COL_A: track 184.0 -> 182.6 mm
Other:
- board size 418.9 x 150.2 mm -> 419 x 150.2 mm

Commit message: push fix rev 1
Routing:
- net ROW_8: track 566.2 -> 847.1 mm
- net GND: track 19.8 -> 5.39 mm, vias 6 -> 2
- net unconnected-(SW_26-PadREF): track 0.00 -> 3.64 mm
- net ROW_5: track 850.3 -> 851.0 mm
