File: FXTal_rev1.kicad_pcb (KiCad board)
At the start: 2 copper layers, 419 x 150.2 mm, 118 parts, among them J1 CONN_CAP_IBM_F

Commit message: push
Other:
- board text added: "FXTal Rev. 1 #: 0"
- board text removed: "FXTal Rev. 2 #: 0"
